Commit message: working wiz + fingers

File: urdf/onrobot_2fg14.xacro (robot description, xacro)
@@ -55,5 +55,5 @@
       </inertial>
       <visual>
-        <origin xyz="-0.032239 0.029494 -0.12005" rpy="0 0 0"/>
+        <origin xyz="0.054361 -0.029494 -0.12005" rpy="0 0 0"/>
         <geometry>
           <mesh filename="package://ur_onrobot/meshes/left_finger_link.stl" scale="0.001 0.001 0.001"/>
@@ -62,5 +62,5 @@
       </visual>
       <collision name="left_finger_collision">
-        <origin xyz="-0.032239 0.029494 -0.12005" rpy="0 0 0"/>
+        <origin xyz="0.054361 -0.029494 -0.12005" rpy="0 0 0"/>
         <geometry>
           <mesh filename="package://ur_onrobot/meshes/left_finger_link.stl" scale="0.001 0.001 0.001"/>
@@ -69,8 +69,8 @@
     </link>
     <joint name="${prefix}left_finger_joint" type="prismatic">
-      <origin xyz="0.032239 -0.029494 0.12005" rpy="0 0 0"/>
+      <origin xyz="-0.054361 0.029494 0.12005" rpy="0 0 0"/>
       <parent link="${prefix}base_link"/>
       <child link="${prefix}left_finger_link"/>
-      <axis xyz="-1.0 0.0 0.0"/>
+      <axis xyz="1.0 0.0 0.0"/>
       <!-- FG14: 0-140mm stroke = 0.070m per finger (vs FG7: 0.019m) -->
       <limit lower="0.0" upper="0.070" effort="300" velocity="0.45"/>
@@ -80,5 +80,5 @@
       <parent link="${prefix}base_link"/>
       <child link="${prefix}right_finger_link"/>
-      <axis xyz="1.0 0.0 0.0"/>
+      <axis xyz="-1.0 0.0 0.0"/>
       <!-- Symmetric movement with mimic joint -->
       <limit lower="-0.070" upper="0.070" effort="300" velocity="0.45"/>
@@ -114,5 +114,5 @@
       </inertial>
       <visual>
-        <origin xyz="0.054361 0.029494 -0.12005" rpy="0 0 0"/>
+        <origin xyz="0.04 0.029494 -0.1199" rpy="0 0 0"/>
         <geometry>
           <mesh filename="package://ur_onrobot/meshes/right_finger_link.stl" scale="0.001 0.001 0.001"/>
@@ -121,5 +121,5 @@
       </visual>
       <collision>
-        <origin xyz="0.054361 0.029494 -0.12005" rpy="0 0 0"/>
+        <origin xyz="0.04 0.029494 -0.1199" rpy="0 0 0"/>
         <geometry>
           <mesh filename="package://ur_onrobot/meshes/right_finger_link.stl" scale="0.001 0.001 0.001"/>
@@ -134,5 +134,5 @@
       </inertial>
       <visual>
-        <origin xyz="-0.032239 0.029494 -0.12005" rpy="0 0 0"/>
+        <origin xyz="-0.04 0.029494 -0.1199" rpy="0 0 0"/>
         <geometry>
           <mesh filename="package://ur_onrobot/meshes/left_finger_link.stl" scale="0.001 0.001 0.001"/>
@@ -141,5 +141,5 @@
       </visual>
       <collision>
-        <origin xyz="-0.032239 0.029494 -0.12005" rpy="0 0 0"/>
+        <origin xyz="-0.04 0.029494 -0.1199" rpy="0 0 0"/>
         <geometry>
           <mesh filename="package://ur_onrobot/meshes/left_finger_link.stl" scale="0.001 0.001 0.001"/>
@@ -148,5 +148,6 @@
     </link>
     <joint name="${prefix}left_finger_joint" type="prismatic">
-      <origin xyz="0.032239 -0.029494 0.12005" rpy="0 0 0"/>
+      <origin xyz="0 -0.029494 0.12005" rpy="0 0 0"/>
+      <!-- <origin xyz="0.032239 -0.029494 0.12005" rpy="0 0 0"/> -->
       <parent link="${prefix}base_link"/>
       <child link="${prefix}left_finger_link"/>
@@ -155,5 +156,7 @@
     </joint>
     <joint name="${prefix}right_finger_joint" type="prismatic">
-      <origin xyz="-0.054361 -0.029494 0.12005" rpy="0 0 0"/>
+      <origin xyz="0 -0.029494 0.12005" rpy="0 0 0"/>
+      <!-- good -0.02 -->
+      <!-- <origin xyz="-0.054361 -0.029494 0.12005" rpy="0 0 0"/> -->
       <parent link="${prefix}base_link"/>
       <child link="${prefix}right_finger_link"/>
@@ -164,8 +167,3 @@
   </xacro:if>
 </xacro:macro>
-<!-- Default parameters for standalone visualization -->
-<xacro:arg name="prefix" default=""/>
-<xacro:arg name="finger_configuration" default="outwards"/>
-<!-- Instantiate the gripper by default for standalone visualization -->
-<xacro:onrobot_2fg14_gripper prefix="$(arg prefix)" finger_configuration="$(arg finger_configuration)"/>
 </robot>

Commit message: Add SRDF configuration for gripper joints and disable collisions

File: urdf/onrobot_2fg14.xacro (robot description, xacro)
@@ -21,10 +21,4 @@
         <material name="silver"/>
       </visual>
-      <collision>
-        <origin xyz="0 0 0" rpy="0 0 0"/>
-        <geometry>
-          <mesh filename="package://ur_onrobot/meshes/base_link.stl" scale="0.001 0.001 0.001"/>
-        </geometry>
-      </collision>
     </link>
     <link name="${prefix}right_finger_link">
@@ -41,10 +35,4 @@
         <material name="silver"/>
       </visual>
-      <collision name="right_finger_collision">
-        <origin xyz="0.054361 0.029494 -0.12005" rpy="0 0 0"/>
-        <geometry>
-          <mesh filename="package://ur_onrobot/meshes/right_finger_link.stl" scale="0.001 0.001 0.001"/>
-        </geometry>
-      </collision>
     </link>
     <link name="${prefix}left_finger_link">
@@ -61,10 +49,4 @@
         <material name="silver"/>
       </visual>
-      <collision name="left_finger_collision">
-        <origin xyz="0.054361 -0.029494 -0.12005" rpy="0 0 0"/>
-        <geometry>
-          <mesh filename="package://ur_onrobot/meshes/left_finger_link.stl" scale="0.001 0.001 0.001"/>
-        </geometry>
-      </collision>
     </link>
     <joint name="${prefix}left_finger_joint" type="prismatic">
@@ -100,10 +82,4 @@
         <material name="silver"/>
       </visual>
-      <collision>
-        <origin xyz="0 0 0" rpy="0 0 0"/>
-        <geometry>
-          <mesh filename="package://ur_onrobot/meshes/base_link.stl" scale="0.001 0.001 0.001"/>
-        </geometry>
-      </collision>
     </link>
     <link name="${prefix}right_finger_link">
@@ -114,5 +90,5 @@
       </inertial>
       <visual>
-        <origin xyz="0.04 0.029494 -0.1199" rpy="0 0 0"/>
+        <origin xyz="0.04 0.029494 -0.119" rpy="0 0 0"/>
         <geometry>
           <mesh filename="package://ur_onrobot/meshes/right_finger_link.stl" scale="0.001 0.001 0.001"/>
@@ -120,10 +96,4 @@
         <material name="silver"/>
       </visual>
-      <collision>
-        <origin xyz="0.04 0.029494 -0.1199" rpy="0 0 0"/>
-        <geometry>
-          <mesh filename="package://ur_onrobot/meshes/right_finger_link.stl" scale="0.001 0.001 0.001"/>
-        </geometry>
-      </collision>
     </link>
     <link name="${prefix}left_finger_link">
@@ -134,5 +104,5 @@
       </inertial>
       <visual>
-        <origin xyz="-0.04 0.029494 -0.1199" rpy="0 0 0"/>
+        <origin xyz="-0.04 0.029494 -0.119" rpy="0 0 0"/>
         <geometry>
           <mesh filename="package://ur_onrobot/meshes/left_finger_link.stl" scale="0.001 0.001 0.001"/>
@@ -140,10 +110,4 @@
         <material name="silver"/>
       </visual>
-      <collision>
-        <origin xyz="-0.04 0.029494 -0.1199" rpy="0 0 0"/>
-        <geometry>
-          <mesh filename="package://ur_onrobot/meshes/left_finger_link.stl" scale="0.001 0.001 0.001"/>
-        </geometry>
-      </collision>
     </link>
     <joint name="${prefix}left_finger_joint" type="prismatic">

Commit message: Add collision geometries and update materials for gripper links

File: urdf/onrobot_2fg14.xacro (robot description, xacro)
@@ -21,4 +21,10 @@
         <material name="silver"/>
       </visual>
+      <collision>
+        <origin xyz="0 0 0.05" rpy="0 0 0"/>
+        <geometry>
+          <box size="0.5 0.5 0.06"/>
+        </geometry>
+      </collision>
     </link>
     <link name="${prefix}right_finger_link">
@@ -33,6 +39,12 @@
           <mesh filename="package://ur_onrobot/meshes/right_finger_link.stl" scale="0.001 0.001 0.001"/>
         </geometry>
-        <material name="silver"/>
+        <material name="black"/>
       </visual>
+      <collision>
+        <origin xyz="0.04 0 0" rpy="0 0 0"/>
+        <geometry>
+          <box size="0.02 0.012 0.05"/>
+        </geometry>
+      </collision>
     </link>
     <link name="${prefix}left_finger_link">
@@ -47,6 +59,12 @@
           <mesh filename="package://ur_onrobot/meshes/left_finger_link.stl" scale="0.001 0.001 0.001"/>
         </geometry>
-        <material name="silver"/>
+        <material name="black"/>
       </visual>
+      <collision>
+        <origin xyz="0.04 0 0" rpy="0 0 0"/>
+        <geometry>
+          <box size="0.02 0.012 0.05"/>
+        </geometry>
+      </collision>
     </link>
     <joint name="${prefix}left_finger_joint" type="prismatic">
@@ -82,4 +100,10 @@
         <material name="silver"/>
       </visual>
+      <collision>
+        <origin xyz="0 0 0.05" rpy="0 0 0"/>
+        <geometry>
+          <box size="0.05 0.05 0.06"/>
+        </geometry>
+      </collision>
     </link>
     <link name="${prefix}right_finger_link">
@@ -94,6 +118,14 @@
           <mesh filename="package://ur_onrobot/meshes/right_finger_link.stl" scale="0.001 0.001 0.001"/>
         </geometry>
-        <material name="silver"/>
+        <material name="red_silver">
+          <color rgba="0.8 0.5 0.5 1"/>
+        </material>
       </visual>
+      <collision>
+        <origin xyz="0.01 0.029494 0.025" rpy="0 0 0"/>
+        <geometry>
+          <box size="0.004 0.02 0.05"/>
+        </geometry>
+      </collision>
     </link>
     <link name="${prefix}left_finger_link">
@@ -110,4 +142,10 @@
         <material name="silver"/>
       </visual>
+      <collision>
+        <origin xyz="-0.01 0.029494 0.025" rpy="0 0 0"/>
+        <geometry>
+          <box size="0.004 0.02 0.05"/>
+        </geometry>
+      </collision>
     </link>
     <joint name="${prefix}left_finger_joint" type="prismatic">
