Commit message: Enhance URDF configuration: add base parameters and update joint definitions for robot mounting

File: urdf/ur_with_onrobot_generic.xacro (robot description, xacro)
@@ -1,4 +1,4 @@
 <?xml version="1.0"?>
-<robot xmlns:xacro="http://www.ros.org/wiki/xacro">
+<robot name="ur" xmlns:xacro="http://www.ros.org/wiki/xacro">
   <!-- Generic UR + OnRobot URDF (works without binary patches) -->
   <!-- Uses name="ur" by default → creates ur_manipulator planning group -->
@@ -18,4 +18,10 @@
   <xacro:arg name="ur_type" default="ur10e"/>
   <xacro:arg name="prefix" default=""/>
+  <xacro:arg name="base_x" default="0.0"/>
+  <xacro:arg name="base_y" default="0.0"/>
+  <xacro:arg name="base_z" default="0.0"/>
+  <xacro:arg name="base_roll" default="0.0"/>
+  <xacro:arg name="base_pitch" default="0.0"/>
+  <xacro:arg name="base_yaw" default="0.0"/>
   <xacro:arg name="use_fake_hardware" default="false"/>
   <xacro:arg name="fake_sensor_commands" default="false"/>
@@ -52,4 +58,12 @@
   <!-- World link for robot attachment -->
   <link name="world"/>
+  <link name="$(arg tf_prefix)robot_mount"/>
+  <joint name="base_to_robot_mount" type="fixed">
+    <parent link="world"/>
+    <child link="$(arg tf_prefix)robot_mount"/>
+    <origin
+      xyz="$(arg base_x) $(arg base_y) $(arg base_z)"
+      rpy="$(arg base_roll) $(arg base_pitch) $(arg base_yaw)" />
+  </joint>
   <!-- Convert args to properties for use in macro -->
   <xacro:property name="initial_positions_file_prop" default="$(arg initial_positions_file)"/>
@@ -58,5 +72,5 @@
     name="$(arg name)"
     tf_prefix="$(arg tf_prefix)"
-    parent="world"
+    parent="$(arg tf_prefix)robot_mount"
     joint_limits_parameters_file="$(arg joint_limit_params)"
     kinematics_parameters_file="$(arg kinematics_params)"
@@ -94,5 +108,5 @@
     keep_alive_count="$(arg keep_alive_count)"
   >
-    <origin xyz="0 0 0" rpy="0 0 0" />
+  <origin xyz="0 0 0" rpy="0 0 0" />
   </xacro:ur_robot>
   <!-- Include OnRobot gripper macro -->
@@ -106,5 +120,5 @@
   </joint>
   <!-- add camera -->
-  <link name="camera_link">
+  <link name="$(arg tf_prefix)camera_link">
     <visual>
       <origin xyz="0 0 0" rpy="0 0 0"/>
@@ -118,7 +132,7 @@
   </link>
   <!-- Joint to attach camera to world (adjust parent/origin as needed) -->
-  <joint name="camera_joint" type="fixed">
+  <joint name="$(arg tf_prefix)camera_joint" type="fixed">
     <parent link="$(arg tf_prefix)tool0"/>
-    <child link="camera_link"/>
+    <child link="$(arg tf_prefix)camera_link"/>
     <origin xyz="0.0 -0.04 0.11" rpy="0 0 0"/>
   </joint>

Commit message: Add collision geometry for camera attachment in URDF

File: urdf/ur_with_onrobot_generic.xacro (robot description, xacro)
@@ -130,4 +130,10 @@
       </material>
     </visual>
+    <collision>
+      <origin xyz="0 0 0" rpy="0 0 0"/>
+      <geometry>
+        <box size="0.05 0.015 0.015"/>
+      </geometry>
+    </collision>
   </link>
   <!-- Joint to attach camera to world (adjust parent/origin as needed) -->

Commit message: move cam 2cm back

File: urdf/ur_with_onrobot_generic.xacro (robot description, xacro)
@@ -141,5 +141,5 @@
     <parent link="$(arg tf_prefix)tool0"/>
     <child link="$(arg tf_prefix)camera_link"/>
-    <origin xyz="0.0 -0.04 0.11" rpy="0 0 0"/>
+    <origin xyz="0.0 -0.04 0.09" rpy="0 0 0"/>
   </joint>
   <!-- Instantiate gripper (will create gripper_prefix + base_link, left_finger_link, right_finger_link) -->

Commit message: cam move up

File: urdf/ur_with_onrobot_generic.xacro (robot description, xacro)
@@ -141,5 +141,5 @@
     <parent link="$(arg tf_prefix)tool0"/>
     <child link="$(arg tf_prefix)camera_link"/>
-    <origin xyz="0.0 -0.04 0.09" rpy="0 0 0"/>
+    <origin xyz="0.0 -0.065 0.09" rpy="0 0 0"/>
   </joint>
   <!-- Instantiate gripper (will create gripper_prefix + base_link, left_finger_link, right_finger_link) -->
